Commit message: Improved demo

File: rrbot_description/urdf/rrbot.tutorial.xacro (robot description, xacro)
@@ -1,5 +1,7 @@
 <?xml version="1.0"?>
 <!-- Revolute-Revolute Manipulator -->
-<robot name="rrbot" xmlns:xacro="http://www.ros.org/wiki/xacro">
+<robot name="rrbot"
+  xmlns:xacro="http://www.ros.org/wiki/xacro"
+  xmlns:controller="http://playerstage.sourceforge.net/gazebo/xmlschema/#controller">
   <xacro:property name="PI" value="3.1415926535897931"/>
   <xacro:property name="width" value="0.1" />
@@ -8,6 +10,4 @@
   <xacro:property name="height3" value="1" />
   <xacro:property name="axel_offset" value="0.05" />
-  <include filename="$(find rrbot_description)/urdf/rrbot.gazebo" />
-  <include filename="$(find rrbot_description)/urdf/materials.xacro" />
   <link name="world"/>
   <link name="link1">
@@ -23,5 +23,7 @@
 	<box size="${width} ${width} ${height1}"/>
       </geometry>
-      <material name="orange"/>
+      <material name="red">
+	<color rgba="0.6 0 0 1.0"/>
+      </material>
     </visual>
     <inertial>
@@ -46,5 +48,7 @@
 	<box size="${width} ${width} ${height2}"/>
       </geometry>
-      <material name="black"/>
+      <material name="green">
+	<color rgba="0 0.6 0 1.0"/>
+      </material>
     </visual>
     <inertial>
@@ -69,5 +73,7 @@
 	<box size="${width} ${width} ${height3}"/>
       </geometry>
-      <material name="orange"/>
+      <material name="blue">
+	<color rgba="0 0 0.6 1.0"/>
+      </material>
     </visual>
     <inertial>
