Commit message: Removed tutorial versions

File: rrbot_description/urdf/rrbot.xacro (robot description, xacro)
@@ -2,13 +2,22 @@
 <!-- Revolute-Revolute Manipulator -->
 <robot name="rrbot" xmlns:xacro="http://www.ros.org/wiki/xacro">
+  <!-- Constants for robot dimensions -->
   <xacro:property name="PI" value="3.1415926535897931"/>
-  <xacro:property name="width" value="0.1" />
-  <xacro:property name="height1" value="2" />
-  <xacro:property name="height2" value="1" />
-  <xacro:property name="height3" value="1" />
-  <xacro:property name="axel_offset" value="0.05" />
+  <xacro:property name="width" value="0.1" /> <!-- Square dimensions (widthxwidth) of beams -->
+  <xacro:property name="height1" value="2" /> <!-- Link 1 -->
+  <xacro:property name="height2" value="1" /> <!-- Link 2 -->
+  <xacro:property name="height3" value="1" /> <!-- Link 3 -->
+  <xacro:property name="axel_offset" value="0.05" /> <!-- Space btw top of beam and the each joint -->
+  <!-- Import all Gazebo-customization elements, including Gazebo colors -->
   <include filename="$(find rrbot_description)/urdf/rrbot.gazebo" />
+  <!-- Import Rviz colors -->
   <include filename="$(find rrbot_description)/urdf/materials.xacro" />
+  <!-- Used for fixing robot to Gazebo 'base_link' -->
   <link name="world"/>
+  <joint name="fixed" type="fixed">
+    <parent link="world"/>
+    <child link="link1"/>
+  </joint>
+  <!-- Base Link -->
   <link name="link1">
     <collision>
@@ -34,4 +43,12 @@
     </inertial>
   </link>
+  <joint name="joint1" type="continuous">
+    <parent link="link1"/>
+    <child link="link2"/>
+    <origin xyz="0 ${width} ${height1 - axel_offset}" rpy="0 0 0"/>
+    <axis xyz="0 1 0"/>
+    <dynamics damping="0.7"/>
+  </joint>
+  <!-- Middle Link -->
   <link name="link2">
     <collision>
@@ -57,4 +74,12 @@
     </inertial>
   </link>
+  <joint name="joint2" type="continuous">
+    <parent link="link2"/>
+    <child link="link3"/>
+    <origin xyz="0 ${width} ${height2 - axel_offset*2}" rpy="0 0 0"/>
+    <axis xyz="0 1 0"/>
+    <dynamics damping="0.7"/>
+  </joint>
+  <!-- Top Link -->
   <link name="link3">
     <collision>
@@ -80,21 +105,3 @@
     </inertial>
   </link>
-  <joint name="fixed" type="fixed">
-    <parent link="world"/>
-    <child link="link1"/>
-  </joint>
-  <joint name="joint1" type="continuous">
-    <parent link="link1"/>
-    <child link="link2"/>
-    <origin xyz="0 ${width} ${height1 - axel_offset}" rpy="0 0 0"/>
-    <axis xyz="0 1 0"/>
-    <dynamics damping="0.7"/>
-  </joint>
-  <joint name="joint2" type="continuous">
-    <parent link="link2"/>
-    <child link="link3"/>
-    <origin xyz="0 ${width} ${height2 - axel_offset*2}" rpy="0 0 0"/>
-    <axis xyz="0 1 0"/>
-    <dynamics damping="0.7"/>
-  </joint>
 </robot>

Commit message: Moved plugin out of rrbot_gazebo

File: rrbot_description/urdf/rrbot.xacro (robot description, xacro)
@@ -35,5 +35,5 @@
     </visual>
     <inertial>
-      <origin xyz="0 0 1" rpy="0 0 0"/>
+      <origin xyz="0 0 ${height1/2}" rpy="0 0 0"/>
       <mass value="1"/>
       <inertia

Commit message: Added sensor plugins

File: rrbot_description/urdf/rrbot.xacro (robot description, xacro)
@@ -8,9 +8,10 @@
   <xacro:property name="height2" value="1" /> <!-- Link 2 -->
   <xacro:property name="height3" value="1" /> <!-- Link 3 -->
+  <xacro:property name="camera_link" value="0.05" /> <!-- Size of square 'camera' box -->
   <xacro:property name="axel_offset" value="0.05" /> <!-- Space btw top of beam and the each joint -->
   <!-- Import all Gazebo-customization elements, including Gazebo colors -->
-  <include filename="$(find rrbot_description)/urdf/rrbot.gazebo" />
+  <xacro:include filename="$(find rrbot_description)/urdf/rrbot.gazebo" />
   <!-- Import Rviz colors -->
-  <include filename="$(find rrbot_description)/urdf/materials.xacro" />
+  <xacro:include filename="$(find rrbot_description)/urdf/materials.xacro" />
   <!-- Used for fixing robot to Gazebo 'base_link' -->
   <link name="world"/>
@@ -105,3 +106,56 @@
     </inertial>
   </link>
+  <joint name="hokuyo_joint" type="fixed">
+    <axis xyz="0 1 0" />
+    <origin xyz="0 0 ${height3 - axel_offset/2}" rpy="0 0 0"/>
+    <parent link="link3"/>
+    <child link="hokuyo_link"/>
+  </joint>
+  <!-- Hokuyo Laser -->
+  <link name="hokuyo_link">
+    <collision>
+      <origin xyz="0 0 0" rpy="0 0 0"/>
+      <geometry>
+	<box size="0.1 0.1 0.1"/>
+      </geometry>
+    </collision>
+    <visual>
+      <origin xyz="0 0 0" rpy="0 0 0"/>
+      <geometry>
+        <mesh filename="package://rrbot_description/meshes/hokuyo.dae"/>
+      </geometry>
+    </visual>
+    <inertial>
+      <mass value="1e-5" />
+      <origin xyz="0 0 0" rpy="0 0 0"/>
+      <inertia ixx="1e-6" ixy="0" ixz="0" iyy="1e-6" iyz="0" izz="1e-6" />
+    </inertial>
+  </link>
+  <joint name="camera_joint" type="fixed">
+    <axis xyz="0 1 0" />
+    <origin xyz="${camera_link} 0 ${height3 - axel_offset*2}" rpy="0 0 0"/>
+    <parent link="link3"/>
+    <child link="camera_link"/>
+  </joint>
+  <!-- Camera -->
+  <link name="camera_link">
+    <collision>
+      <origin xyz="0 0 0" rpy="0 0 0"/>
+      <geometry>
+	<box size="${camera_link} ${camera_link} ${camera_link}"/>
+      </geometry>
+    </collision>
+    <visual>
+      <origin xyz="0 0 0" rpy="0 0 0"/>
+      <geometry>
+	<box size="${camera_link} ${camera_link} ${camera_link}"/>
+      </geometry>
+      <material name="red"/>
+    </visual>
+    <inertial>
+      <mass value="1e-5" />
+      <origin xyz="0 0 0" rpy="0 0 0"/>
+      <inertia ixx="1e-6" ixy="0" ixz="0" iyy="1e-6" iyz="0" izz="1e-6" />
+    </inertial>
+  </link>
 </robot>

Commit message: Integrating ros_control

File: rrbot_description/urdf/rrbot.xacro (robot description, xacro)
@@ -39,7 +39,7 @@
       <mass value="1"/>
       <inertia
-        ixx="1.0" ixy="0.0" ixz="0.0"
-        iyy="1.0" iyz="0.0"
-        izz="1.0"/>
+	  ixx="1.0" ixy="0.0" ixz="0.0"
+	  iyy="1.0" iyz="0.0"
+	  izz="1.0"/>
     </inertial>
   </link>
@@ -70,7 +70,7 @@
       <mass value="1"/>
       <inertia
-        ixx="1.0" ixy="0.0" ixz="0.0"
-        iyy="1.0" iyz="0.0"
-        izz="1.0"/>
+	  ixx="1.0" ixy="0.0" ixz="0.0"
+	  iyy="1.0" iyz="0.0"
+	  izz="1.0"/>
     </inertial>
   </link>
@@ -101,7 +101,7 @@
       <mass value="1"/>
       <inertia
-        ixx="1.0" ixy="0.0" ixz="0.0"
-        iyy="1.0" iyz="0.0"
-        izz="1.0"/>
+	  ixx="1.0" ixy="0.0" ixz="0.0"
+	  iyy="1.0" iyz="0.0"
+	  izz="1.0"/>
     </inertial>
   </link>
@@ -159,3 +159,13 @@
     </inertial>
   </link>
+  <!--transmission name="joint1_trans" type="pr2_mechanism_model/SimpleTransmission">
+    <actuator name="joint1_motor"/>
+    <joint name="joint1"/>
+    <mechanicalReduction>1</mechanicalReduction>
+  </transmission>
+  <transmission name="joint2_trans" type="pr2_mechanism_model/SimpleTransmission">
+    <actuator name="joint2_motor"/>
+    <joint name="joint2"/>
+    <mechanicalReduction>1</mechanicalReduction>
+  </transmission-->
 </robot>

Commit message: use velocity controllers

File: rrbot_description/urdf/rrbot.xacro (robot description, xacro)
@@ -167,11 +167,3 @@
     </actuator>
   </transmission>
-  <transmission name="tran2">
-    <type>transmission_interface/SimpleTransmission</type>
-    <joint name="joint2"/>
-    <actuator name="motor2">
-      <hardwareInterface>VelocityJointInterface</hardwareInterface>
-      <mechanicalReduction>1</mechanicalReduction>
-    </actuator>
-  </transmission>
 </robot>

Commit message: fix hardware interface controller error missing for joint1

File: rrbot_description/urdf/rrbot.xacro (robot description, xacro)
@@ -161,5 +161,7 @@
   <transmission name="tran1">
     <type>transmission_interface/SimpleTransmission</type>
-    <joint name="joint1"/>
+    <joint name="joint1">
+      <hardwareInterface>EffortJointInterface</hardwareInterface>
+    </joint>
     <actuator name="motor1">
       <hardwareInterface>EffortJointInterface</hardwareInterface>

Commit message: add hardwareinterface to joint in transmission tag

File: rrbot_description/urdf/rrbot.xacro (robot description, xacro)
@@ -161,5 +161,7 @@
   <transmission name="tran1">
     <type>transmission_interface/SimpleTransmission</type>
-    <joint name="joint1"/>
+    <joint name="joint1">
+      <hardwareInterface>EffortJointInterface</hardwareInterface>
+    </joint>
     <actuator name="motor1">
       <hardwareInterface>EffortJointInterface</hardwareInterface>
@@ -169,5 +171,7 @@
   <transmission name="tran2">
     <type>transmission_interface/SimpleTransmission</type>
-    <joint name="joint2"/>
+    <joint name="joint2">
+      <hardwareInterface>EffortJointInterface</hardwareInterface>
+    </joint>
     <actuator name="motor2">
       <hardwareInterface>EffortJointInterface</hardwareInterface>

Commit message: rrbot_description: improve inertia values
The current inertia matrix values don't match
the geometry of the robot.
This auto-calculates the ixx,iyy,izz values
based on the arbitrary mass value of 1.0
The mass is still arbitrary, but now the
inertia values should be geometrically
consistent.

File: rrbot_description/urdf/rrbot.xacro (robot description, xacro)
@@ -4,4 +4,5 @@
   <!-- Constants for robot dimensions -->
   <xacro:property name="PI" value="3.1415926535897931"/>
+  <xacro:property name="mass" value="1" /> <!-- arbitrary value for mass -->
   <xacro:property name="width" value="0.1" /> <!-- Square dimensions (widthxwidth) of beams -->
   <xacro:property name="height1" value="2" /> <!-- Link 1 -->
@@ -37,9 +38,9 @@
     <inertial>
       <origin xyz="0 0 ${height1/2}" rpy="0 0 0"/>
-      <mass value="1"/>
+      <mass value="${mass}"/>
       <inertia
-	  ixx="1.0" ixy="0.0" ixz="0.0"
-	  iyy="1.0" iyz="0.0"
-	  izz="1.0"/>
+	  ixx="${mass / 12.0 * (width*width + height1*height1)}" ixy="0.0" ixz="0.0"
+	  iyy="${mass / 12.0 * (height1*height1 + width*width)}" iyz="0.0"
+	  izz="${mass / 12.0 * (width*width + width*width)}"/>
     </inertial>
   </link>
@@ -68,9 +69,9 @@
     <inertial>
       <origin xyz="0 0 ${height2/2 - axel_offset}" rpy="0 0 0"/>
-      <mass value="1"/>
+      <mass value="${mass}"/>
       <inertia
-	  ixx="1.0" ixy="0.0" ixz="0.0"
-	  iyy="1.0" iyz="0.0"
-	  izz="1.0"/>
+	  ixx="${mass / 12.0 * (width*width + height2*height2)}" ixy="0.0" ixz="0.0"
+	  iyy="${mass / 12.0 * (height2*height2 + width*width)}" iyz="0.0"
+	  izz="${mass / 12.0 * (width*width + width*width)}"/>
     </inertial>
   </link>
@@ -99,9 +100,9 @@
     <inertial>
       <origin xyz="0 0 ${height3/2 - axel_offset}" rpy="0 0 0"/>
-      <mass value="1"/>
+      <mass value="${mass}"/>
       <inertia
-	  ixx="1.0" ixy="0.0" ixz="0.0"
-	  iyy="1.0" iyz="0.0"
-	  izz="1.0"/>
+	  ixx="${mass / 12.0 * (width*width + height3*height3)}" ixy="0.0" ixz="0.0"
+	  iyy="${mass / 12.0 * (height3*height3 + width*width)}" iyz="0.0"
+	  izz="${mass / 12.0 * (width*width + width*width)}"/>
     </inertial>
   </link>

Commit message: Test branch that includes screen display

File: rrbot_description/urdf/rrbot.xacro (robot description, xacro)
@@ -160,4 +160,26 @@
     </inertial>
   </link>
+  <joint name="display_joint" type="fixed">
+    <origin rpy="0 0 0" xyz="0.0 -0.016 0.0"/>
+    <parent link="link3"/>
+    <child link="display"/>
+  </joint>
+  <!-- Screen Display -->
+  <link name="display">
+    <visual>
+      <origin rpy="0.2617993877991494 0 0" xyz="0 0 0"/>
+      <geometry>
+        <box size="0.218 0.16 0.001"/>
+      </geometry>
+      <material name="black">
+        <color rgba="0 0 0 1"/>
+      </material>
+    </visual>
+    <inertial>
+      <origin rpy="0 0 0" xyz="0 0 0"/>
+      <mass value="0.0001"/>
+      <inertia ixx="1e-08" ixy="0" ixz="0" iyy="1e-08" iyz="0" izz="1e-08"/>
+    </inertial>
+  </link>
   <transmission name="tran1">
     <type>transmission_interface/SimpleTransmission</type>

Commit message: beautify xacro
Signed-off-by: ahcorde <ahcorde@gmail.com>

File: rrbot_description/urdf/rrbot.xacro (robot description, xacro)
@@ -4,15 +4,22 @@
   <!-- Constants for robot dimensions -->
   <xacro:property name="PI" value="3.1415926535897931"/>
-  <xacro:property name="mass" value="1" /> <!-- arbitrary value for mass -->
-  <xacro:property name="width" value="0.1" /> <!-- Square dimensions (widthxwidth) of beams -->
-  <xacro:property name="height1" value="2" /> <!-- Link 1 -->
-  <xacro:property name="height2" value="1" /> <!-- Link 2 -->
-  <xacro:property name="height3" value="1" /> <!-- Link 3 -->
-  <xacro:property name="camera_link" value="0.05" /> <!-- Size of square 'camera' box -->
-  <xacro:property name="axel_offset" value="0.05" /> <!-- Space btw top of beam and the each joint -->
+  <!-- arbitrary value for mass -->
+  <xacro:property name="mass" value="1"/>
+  <!-- Square dimensions (widthxwidth) of beams -->
+  <xacro:property name="width" value="0.1"/>
+  <!-- Link 1 -->
+  <xacro:property name="height1" value="2"/>
+  <!-- Link 2 -->
+  <xacro:property name="height2" value="1"/>
+  <!-- Link 3 -->
+  <xacro:property name="height3" value="1"/>
+  <!-- Size of square 'camera' box -->
+  <xacro:property name="camera_link" value="0.05"/>
+  <!-- Space btw top of beam and the each joint -->
+  <xacro:property name="axel_offset" value="0.05"/>
   <!-- Import all Gazebo-customization elements, including Gazebo colors -->
-  <xacro:include filename="$(find rrbot_description)/urdf/rrbot.gazebo" />
+  <xacro:include filename="$(find rrbot_description)/urdf/rrbot.gazebo"/>
   <!-- Import Rviz colors -->
-  <xacro:include filename="$(find rrbot_description)/urdf/materials.xacro" />
+  <xacro:include filename="$(find rrbot_description)/urdf/materials.xacro"/>
   <!-- Used for fixing robot to Gazebo 'base_link' -->
   <link name="world"/>
@@ -26,5 +33,5 @@
       <origin xyz="0 0 ${height1/2}" rpy="0 0 0"/>
       <geometry>
-	       <box size="${width} ${width} ${height1}"/>
+        <box size="${width} ${width} ${height1}"/>
       </geometry>
     </collision>
@@ -32,5 +39,5 @@
       <origin xyz="0 0 ${height1/2}" rpy="0 0 0"/>
       <geometry>
-	       <box size="${width} ${width} ${height1}"/>
+        <box size="${width} ${width} ${height1}"/>
       </geometry>
       <material name="orange"/>
@@ -39,8 +46,5 @@
       <origin xyz="0 0 ${height1/2}" rpy="0 0 0"/>
       <mass value="${mass}"/>
-      <inertia
-	  ixx="${mass / 12.0 * (width*width + height1*height1)}" ixy="0.0" ixz="0.0"
-	  iyy="${mass / 12.0 * (height1*height1 + width*width)}" iyz="0.0"
-	  izz="${mass / 12.0 * (width*width + width*width)}"/>
+      <inertia ixx="${mass / 12.0 * (width*width + height1*height1)}" ixy="0.0" ixz="0.0" iyy="${mass / 12.0 * (height1*height1 + width*width)}" iyz="0.0" izz="${mass / 12.0 * (width*width + width*width)}"/>
     </inertial>
   </link>
@@ -57,5 +61,5 @@
       <origin xyz="0 0 ${height2/2 - axel_offset}" rpy="0 0 0"/>
       <geometry>
-	       <box size="${width} ${width} ${height2}"/>
+        <box size="${width} ${width} ${height2}"/>
       </geometry>
     </collision>
@@ -63,5 +67,5 @@
       <origin xyz="0 0 ${height2/2 - axel_offset}" rpy="0 0 0"/>
       <geometry>
-	       <box size="${width} ${width} ${height2}"/>
+        <box size="${width} ${width} ${height2}"/>
       </geometry>
       <material name="black"/>
@@ -70,8 +74,5 @@
       <origin xyz="0 0 ${height2/2 - axel_offset}" rpy="0 0 0"/>
       <mass value="${mass}"/>
-      <inertia
-	  ixx="${mass / 12.0 * (width*width + height2*height2)}" ixy="0.0" ixz="0.0"
-	  iyy="${mass / 12.0 * (height2*height2 + width*width)}" iyz="0.0"
-	  izz="${mass / 12.0 * (width*width + width*width)}"/>
+      <inertia ixx="${mass / 12.0 * (width*width + height2*height2)}" ixy="0.0" ixz="0.0" iyy="${mass / 12.0 * (height2*height2 + width*width)}" iyz="0.0" izz="${mass / 12.0 * (width*width + width*width)}"/>
     </inertial>
   </link>
@@ -88,5 +89,5 @@
       <origin xyz="0 0 ${height3/2 - axel_offset}" rpy="0 0 0"/>
       <geometry>
-	       <box size="${width} ${width} ${height3}"/>
+        <box size="${width} ${width} ${height3}"/>
       </geometry>
     </collision>
@@ -94,5 +95,5 @@
       <origin xyz="0 0 ${height3/2 - axel_offset}" rpy="0 0 0"/>
       <geometry>
-	       <box size="${width} ${width} ${height3}"/>
+        <box size="${width} ${width} ${height3}"/>
       </geometry>
       <material name="orange"/>
@@ -101,12 +102,9 @@
       <origin xyz="0 0 ${height3/2 - axel_offset}" rpy="0 0 0"/>
       <mass value="${mass}"/>
-      <inertia
-	  ixx="${mass / 12.0 * (width*width + height3*height3)}" ixy="0.0" ixz="0.0"
-	  iyy="${mass / 12.0 * (height3*height3 + width*width)}" iyz="0.0"
-	  izz="${mass / 12.0 * (width*width + width*width)}"/>
+      <inertia ixx="${mass / 12.0 * (width*width + height3*height3)}" ixy="0.0" ixz="0.0" iyy="${mass / 12.0 * (height3*height3 + width*width)}" iyz="0.0" izz="${mass / 12.0 * (width*width + width*width)}"/>
     </inertial>
   </link>
   <joint name="hokuyo_joint" type="fixed">
-    <axis xyz="0 1 0" />
+    <axis xyz="0 1 0"/>
     <origin xyz="0 0 ${height3 - axel_offset/2}" rpy="0 0 0"/>
     <parent link="link3"/>
@@ -118,5 +116,5 @@
       <origin xyz="0 0 0" rpy="0 0 0"/>
       <geometry>
-	       <box size="0.1 0.1 0.1"/>
+        <box size="0.1 0.1 0.1"/>
       </geometry>
     </collision>
@@ -128,11 +126,11 @@
     </visual>
     <inertial>
-      <mass value="1e-5" />
+      <mass value="1e-5"/>
       <origin xyz="0 0 0" rpy="0 0 0"/>
-      <inertia ixx="1e-6" ixy="0" ixz="0" iyy="1e-6" iyz="0" izz="1e-6" />
+      <inertia ixx="1e-6" ixy="0" ixz="0" iyy="1e-6" iyz="0" izz="1e-6"/>
     </inertial>
   </link>
   <joint name="camera_joint" type="fixed">
-    <axis xyz="0 1 0" />
+    <axis xyz="0 1 0"/>
     <origin xyz="${camera_link} 0 ${height3 - axel_offset*2}" rpy="0 0 0"/>
     <parent link="link3"/>
@@ -144,5 +142,5 @@
       <origin xyz="0 0 0" rpy="0 0 0"/>
       <geometry>
-	       <box size="${camera_link} ${camera_link} ${camera_link}"/>
+        <box size="${camera_link} ${camera_link} ${camera_link}"/>
       </geometry>
     </collision>
@@ -150,25 +148,24 @@
       <origin xyz="0 0 0" rpy="0 0 0"/>
       <geometry>
-	       <box size="${camera_link} ${camera_link} ${camera_link}"/>
+        <box size="${camera_link} ${camera_link} ${camera_link}"/>
       </geometry>
       <material name="red"/>
     </visual>
     <inertial>
-      <mass value="1e-5" />
+      <mass value="1e-5"/>
       <origin xyz="0 0 0" rpy="0 0 0"/>
-      <inertia ixx="1e-6" ixy="0" ixz="0" iyy="1e-6" iyz="0" izz="1e-6" />
+      <inertia ixx="1e-6" ixy="0" ixz="0" iyy="1e-6" iyz="0" izz="1e-6"/>
     </inertial>
   </link>
   <!-- generate an optical frame http://www.ros.org/reps/rep-0103.html#suffix-frames
-      so that ros and opencv can operate on the camera frame correctly -->
+   so that ros and opencv can operate on the camera frame correctly -->
   <joint name="camera_optical_joint" type="fixed">
-    <!-- these values have to be these values otherwise the gazebo camera image
-        won't be aligned properly with the frame it is supposedly originating from -->
+    <!-- these values have to be these values otherwise the gazebo camera image won't
+     be aligned properly with the frame it is supposedly originating from -->
     <origin xyz="0 0 0" rpy="${-pi/2} 0 ${-pi/2}"/>
     <parent link="camera_link"/>
     <child link="camera_link_optical"/>
   </joint>
-  <link name="camera_link_optical">
-  </link>
+  <link name="camera_link_optical"></link>
   <ros2_control name="GazeboSystem" type="system">
     <hardware>
